Commit message: quickstart update with column demo

File: modules/bringup/simulator_bringup/urdf/big_robotic.urdf (robot description, URDF)
Before this commit: robot big_robotic, 3 links, 2 joints
Links:
- added link catch_footprint_link; visual cylinder length=0.001 radius=${catch_radius}
Joints:
- added joint base_footprint__catch_footprint_joint: type fixed, parent base_footprint, child catch_footprint_link, origin xyz=${base_length/2 + catch_radius} 0.0 0.01 rpy=0 0 0
